Commit message: 增加了工具坐标系
增加了第7 link，增加了工具坐标系；修正了之前1 4 6轴旋转方向和机器人实际正方向规定不同的问题。

File: kuka_kr4_description/urdf/kuka_kr4_description.urdf (robot description, URDF)
Before this commit: robot kuka_kr4_description, 7 links, 6 joints
Links:
- removed link link1
- removed link link2
- removed link link3
- removed link link4
- removed link link5
- removed link link6
- added link l1, mass 3.49063221731985; collision mesh filename=package://kuka_kr4_description/meshes/l1.STL; visual mesh filename=package://kuka_kr4_description/meshes/l1.STL
- added link l2, mass 4.73302208355957; collision mesh filename=package://kuka_kr4_description/meshes/l2.STL; visual mesh filename=package://kuka_kr4_description/meshes/l2.STL
- added link l3, mass 2.14150525089968; collision mesh filename=package://kuka_kr4_description/meshes/l3.STL; visual mesh filename=package://kuka_kr4_description/meshes/l3.STL
- added link l4, mass 1.09604091499795; collision mesh filename=package://kuka_kr4_description/meshes/l4.STL; visual mesh filename=package://kuka_kr4_description/meshes/l4.STL
- added link l5, mass 0.54429927248745; collision mesh filename=package://kuka_kr4_description/meshes/l5.STL; visual mesh filename=package://kuka_kr4_description/meshes/l5.STL
- added link l6, mass 0.0338899828627831; collision mesh filename=package://kuka_kr4_description/meshes/l6.STL; visual mesh filename=package://kuka_kr4_description/meshes/l6.STL
- added link tool, mass 0.0154467683293326; collision mesh filename=package://kuka_kr4_description/meshes/tool.STL; visual mesh filename=package://kuka_kr4_description/meshes/tool.STL
- link base_link: mass 6.6366 -> 6.63660865962053
Joints:
- removed joint join2
- removed joint join6
- removed joint joint1
- removed joint joint3
- removed joint joint4
- removed joint joint5
- added joint fixed_joint: type fixed, parent l6, child tool, origin xyz=0.14418 0 -0.018 rpy=3.1416 -1.0472 0, axis 0 0 0, limit lower=0 upper=0 effort=0 velocity=0
- added joint j1: type continuous, parent base_link, child l1, origin xyz=0 0 0.167 rpy=0 0 0, axis 0 0 -1, limit lower=-2.9671 upper=2.9671 effort=50 velocity=1.5708
- added joint j2: type revolute, parent l1, child l2, origin xyz=0 0 0.163 rpy=0 0 0, axis 0 1 0, limit lower=-3.4034 upper=0.6981 effort=50 velocity=1.5708
- added joint j3: type continuous, parent l2, child l3, origin xyz=0 0 0.29 rpy=0 0 0, axis 0 1 0, limit lower=-2.0071 upper=2.618 effort=50 velocity=1.5708
- added joint j4: type continuous, parent l3, child l4, origin xyz=0.16262 0 0.02 rpy=0 0 0, axis -1 0 0, limit lower=-3.2289 upper=3.2289 effort=50 velocity=1.5708
- added joint j5: type continuous, parent l4, child l5, origin xyz=0.14738 0 0 rpy=0 0 0, axis 0 1 0, limit lower=-2.0944 upper=2.0944 effort=50 velocity=1.5708
- added joint j6: type continuous, parent l5, child l6, origin xyz=0.048 0 0 rpy=0 0 0, axis -1 0 0, limit lower=-6.1086 upper=6.1086 effort=50 velocity=1.5708

Commit message: l6坐标系改为工件坐标系

File: kuka_kr4_description/urdf/kuka_kr4_description.urdf (robot description, URDF)
Before this commit: robot kuka_kr4_description, 8 links, 7 joints
Links:
- link l2: mass 4.73302208355957 -> 4.73302208355956
- link l5: mass 0.54429927248745 -> 0.544299272487451
Joints:
- joint fixed_joint: origin xyz=0.14418 0 -0.018 rpy=3.1416 -1.0472 0 -> xyz=0 0 0 rpy=0 0 0
- joint j1: type continuous -> revolute
- joint j3: type continuous -> revolute
- joint j4: type continuous -> revolute
- joint j5: origin xyz=0.14738 0 0 rpy=0 0 0 -> xyz=0.147378544382031 0 0 rpy=0 0 0; type continuous -> revolute
- joint j6: axis -1 0 0 -> -0.86603 0 -0.5; origin xyz=0.048 0 0 rpy=0 0 0 -> xyz=0.19218 0 -0.018 rpy=0 0.5236 0; type continuous -> revolute

Commit message: 目前最新版本的urdf和srdf

File: kuka_kr4_description/urdf/kuka_kr4_description.urdf (robot description, URDF)
Before this commit: robot kuka_kr4_description, 8 links, 7 joints
Links:
- removed link tool
- added link tool2, mass 0.00307725233002518; collision mesh filename=package://kuka_kr4_description/meshes/tool2.STL; visual mesh filename=package://kuka_kr4_description/meshes/tool2.STL
- added link tool_1, mass 0.0123695159993075; collision mesh filename=package://kuka_kr4_description/meshes/tool_1.STL; visual mesh filename=package://kuka_kr4_description/meshes/tool_1.STL
- link l1: mass 3.49063221731985 -> 3.49063221756745
- link l3: mass 2.14150525089968 -> 2.14150525350941
- link l4: mass 1.09604091499795 -> 1.09604091906534
- link l5: mass 0.544299272487451 -> 0.544299272455749
Joints:
- removed joint fixed_joint
- added joint fixed_joint_t1: type fixed, parent l6, child tool_1, origin xyz=0.14418 0 -0.018 rpy=0 0.5236 0, axis 0 0 0, limit lower=0 upper=0 effort=0 velocity=0
- added joint fixed_joint_t2: type fixed, parent tool_1, child tool2, origin xyz=0 0 0 rpy=0 0 0, axis 0 0 0
- joint j6: axis -0.86603 0 -0.5 -> -1 0 0; origin xyz=0.19218 0 -0.018 rpy=0 0.5236 0 -> xyz=0.048 0 0 rpy=0 0 0
